Commit message: 250516_1

File: resources/robots/g1_description/g1_29dof_with_hand.urdf (robot description, URDF)
Before this commit: robot g1_29dof_with_hand, 54 links, 53 joints
Joints:
- joint left_hand_thumb_0_joint: limit lower=-1.04719755 upper=1.04719755 effort=2.45 velocity=3.14 -> lower=-1.04719755 upper=1.04719755 effort=2.45 velocity=6.857
- joint right_hand_thumb_0_joint: limit lower=-1.04719755 upper=1.04719755 effort=2.45 velocity=3.14 -> lower=-1.04719755 upper=1.04719755 effort=2.45 velocity=6.857

File: resources/robots/g1_description/g1_29dof_with_hand_rev_1_0.urdf (robot description, URDF)
Before this commit: robot g1_29dof_with_hand_rev_1_0, 53 links, 52 joints
Joints:
- joint left_hand_thumb_0_joint: limit lower=-1.04719755 upper=1.04719755 effort=2.45 velocity=3.14 -> lower=-1.04719755 upper=1.04719755 effort=2.45 velocity=6.857
- joint right_hand_thumb_0_joint: limit lower=-1.04719755 upper=1.04719755 effort=2.45 velocity=3.14 -> lower=-1.04719755 upper=1.04719755 effort=2.45 velocity=6.857
